Commit message: update dynamic parameters to approximate the bathydrone

File: simulation/boat_model/src/bathyboat/bathyboat_custom.urdf (robot description, URDF)
Before this commit: robot bathydrone, 2 links, 1 joints
Links:
- link wamv/dummy_link: mass 180.0 -> 6.342; geometry collision box size=0.65 0.2 0.1; collision box size=0.65 0.2 0.1

Commit message: update blender to have right COM locationa and add documentation for simulation model

File: simulation/boat_model/src/bathyboat/bathyboat_custom.urdf (robot description, URDF)
Before this commit: robot bathydrone, 2 links, 1 joints
Links:
- link wamv/dummy_link: geometry collision box size=0.65 0.2 0.1; collision box size=0.65 0.2 0.1

File: simulation/boat_model/src/bathyboat_custom.urdf.xacro (robot description, xacro)
@@ -2,5 +2,5 @@
 <robot name="bathydrone" xmlns:xacro="http://ros.org/wiki/xacro">
   <!-- Defines the base vehicle -->
-  <xacro:include filename="$(find vrx_gazebo)/../wamv_description/urdf/wamv_base.urdf.xacro" />
+  <xacro:include filename="$(find boat_model)/src/bathyboat/bathyboat_base.urdf.xacro" />
   <!-- Attach tension and hydrodynamics plugin -->
   <xacro:include filename="include_tension_to_model.xacro"/>
